File: hardware/shd_v1.0.brd (EAGLE design)
At the start: 65.2 x 21.8 mm, 16 parts

Commit message: minor changes and bug fixes
Parts:
- added SJ1: (no value), jumper:SJ_2
Connections:
- new net TMP_ANA: SJ1.1, U1.ADC
- new net TMP_DATA: SJ1.3
- net V_TMP: now also SJ1.2; no longer U1.ADC
Routing:
- net V_TMP: track 38.2 -> 28.7 mm, vias 2 -> 0
- net TMP_ANA: track 0.00 -> 9.39 mm, vias 0 -> 1
- net VDD_3.3: track 59.8 -> 64.8 mm
- net RST: track 48.2 -> 50.0 mm
- net TMP_DATA: track 0.00 -> 1.48 mm, vias 0 -> 1
- net GPIO0: track 30.9 -> 30.4 mm
Changed lines of the file:
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@@
 <?xml version="1.0" encoding="utf-8"?>
 <!DOCTYPE eagle SYSTEM "eagle.dtd">
-<eagle version="9.2.2">
+<eagle version="9.3.0">
 <drawing>
 <settings>
@@
 <attribute name="VALUE" x="14.4894" y="10.615" size="1.27" layer="27" font="vector" ratio="10"/>
 </element>
+<element name="SJ1" library="jumper" library_urn="urn:adsk.eagle:library:252" package="SJ_2" package3d_urn="urn:adsk.eagle:package:15474/1" value="" x="46.5" y="14" smashed="yes" rot="MR0">
+<attribute name="NAME" x="47.913" y="15.77" size="1.27" layer="26" ratio="10" rot="MR0"/>
+<attribute name="VALUE" x="46.6001" y="14" size="0.02" layer="28" rot="MR0"/>
+</element>
 </elements>
 <signals>
@@
 <contactref element="R_RST" pad="1"/>
 <contactref element="U1" pad="RESET"/>
-<wire x1="33.08" y1="13.625" x2="54.75" y2="13.625" width="0.3" layer="16"/>
+<wire x1="54.75" y1="12.375" x2="34.33" y2="12.375" width="0.3" layer="16"/>
 <wire x1="15.02" y1="19" x2="15.02" y2="17.73" width="0.3" layer="16"/>
 <wire x1="55.05" y1="19.05" x2="54.75" y2="18.75" width="0.3" layer="1"/>
-<wire x1="54.75" y1="18.75" x2="54.75" y2="13.625" width="0.3" layer="1"/>
-<via x="54.75" y="13.625" extent="1-16" drill="0.35"/>
+<wire x1="54.75" y1="18.75" x2="54.75" y2="12.375" width="0.3" layer="1"/>
+<via x="54.75" y="12.375" extent="1-16" drill="0.35"/>
 <wire x1="30.625" y1="13.625" x2="33.08" y2="13.625" width="0.3" layer="16"/>
-<wire x1="29.625" y1="14.625" x2="30.625" y2="13.625" width="0.3" layer="16"/>
-<wire x1="29.5" y1="14.75" x2="29.625" y2="14.625" width="0.3" layer="16"/>
+<wire x1="29.5" y1="14.75" x2="30.625" y2="13.625" width="0.3" layer="16"/>
 <wire x1="15.02" y1="17.73" x2="18" y2="14.75" width="0.3" layer="16"/>
 <wire x1="18" y1="14.75" x2="29.5" y2="14.75" width="0.3" layer="16"/>
+<wire x1="34.33" y1="12.375" x2="33.08" y2="13.625" width="0.3" layer="16"/>
 </signal>
 <signal name="VCC_5.0">
@@
 <via x="48.5" y="8" extent="1-16" drill="0.35"/>
 <via x="51.5" y="6.75" extent="1-16" drill="0.35"/>
-<via x="52.75" y="12.25" extent="1-16" drill="0.35"/>
-<via x="48.75" y="12" extent="1-16" drill="0.35"/>
+<via x="53" y="11.5" extent="1-16" drill="0.35"/>
+<via x="49" y="11.25" extent="1-16" drill="0.35"/>
 <via x="38.75" y="17.5" extent="1-16" drill="0.35"/>
 <via x="39" y="19.75" extent="1-16" drill="0.35"/>
@@
 <via x="30.25" y="17.25" extent="1-16" drill="0.35"/>
 <via x="31.5" y="4.25" extent="1-16" drill="0.35"/>
+<via x="22" y="12.5" extent="1-16" drill="0.35"/>
+<wire x1="21" y1="9.25" x2="22" y2="12.5" width="0" layer="19" extent="1-1"/>
 </signal>
 <signal name="VDD_3.3">
@@
 <wire x1="21.67" y1="17.5" x2="19.25" y2="17.5" width="0.5" layer="1"/>
 <wire x1="22.92" y1="16.25" x2="22.92" y2="13.625" width="0.5" layer="1"/>
-<wire x1="35.25" y1="13.05" x2="35.45" y2="13.05" width="0.8" layer="1"/>
-<wire x1="35.45" y1="13.05" x2="36.5" y2="12" width="0.8" layer="1"/>
-<via x="36.5" y="12" extent="1-16" drill="0.35"/>
-<wire x1="36.5" y1="12" x2="42" y2="12" width="0.8" layer="16"/>
-<via x="42" y="12" extent="1-16" drill="0.35"/>
-<wire x1="42" y1="16" x2="42" y2="12" width="0.8" layer="1"/>
+<wire x1="36.5" y1="11.5" x2="35.25" y2="12.75" width="0.8" layer="1"/>
+<wire x1="35.25" y1="13.05" x2="35.25" y2="12.75" width="0.8" layer="1"/>
+<via x="36.5" y="11.5" extent="1-16" drill="0.35"/>
+<wire x1="36.5" y1="11.5" x2="42" y2="11.5" width="0.8" layer="16"/>
+<via x="42" y="11.5" extent="1-16" drill="0.35"/>
+<wire x1="42" y1="11.5" x2="42" y2="16.25" width="0.8" layer="1"/>
 <wire x1="35.25" y1="13.05" x2="34.7" y2="12.5" width="0.5" layer="1"/>
 <wire x1="30.5" y1="13.75" x2="31.75" y2="12.5" width="0.5" layer="1"/>
 <wire x1="34.7" y1="12.5" x2="31.75" y2="12.5" width="0.5" layer="1"/>
-<wire x1="41.05" y1="19.05" x2="41.05" y2="17.2" width="0.8" layer="1"/>
-<wire x1="41.5" y1="16.75" x2="41.5" y2="16.5" width="0.8" layer="1"/>
-<wire x1="41.5" y1="16.75" x2="41.05" y2="17.2" width="0.8" layer="1"/>
-<wire x1="41.5" y1="16.5" x2="42" y2="16" width="0.8" layer="1"/>
-<via x="41.5" y="16.5" extent="1-16" drill="0.35"/>
-<wire x1="41.5" y1="16.5" x2="42" y2="17" width="0.3" layer="16"/>
-<wire x1="42" y1="17" x2="50.75" y2="17" width="0.3" layer="16"/>
+<wire x1="41.05" y1="17.2" x2="41.05" y2="19.05" width="0.8" layer="1"/>
 <wire x1="50.75" y1="17" x2="51" y2="16.75" width="0.3" layer="16"/>
 <via x="51" y="16.75" extent="1-16" drill="0.35"/>
@@
 <wire x1="31.5" y1="16.5" x2="31.5" y2="19" width="0.5" layer="1"/>
 <wire x1="19.25" y1="17.5" x2="18" y2="18.75" width="0.5" layer="1"/>
+<wire x1="42" y1="16.25" x2="41.05" y2="17.2" width="0.8" layer="1"/>
+<wire x1="41.05" y1="19.05" x2="40.75" y2="18.75" width="0.3" layer="1"/>
+<wire x1="40.75" y1="18.75" x2="39.75" y2="18.75" width="0.3" layer="1"/>
+<via x="39.75" y="18.75" extent="1-16" drill="0.35"/>
+<wire x1="39.75" y1="18.75" x2="49" y2="18.75" width="0.3" layer="16"/>
+<wire x1="49" y1="18.75" x2="51" y2="16.75" width="0.3" layer="16"/>
 </signal>
 <signal name="TX">
@@
 <contactref element="R_PROG" pad="1"/>
 <contactref element="U1" pad="GPIO0"/>
-<via x="47.05" y="15.9306" extent="1-16" drill="0.35"/>
-<wire x1="47.05" y1="2.65" x2="47.05" y2="15.9306" width="0.3" layer="1"/>
-<wire x1="47.05" y1="15.9306" x2="46.8218" y2="15.7024" width="0.3" layer="16"/>
-<wire x1="33.6276" y1="15.7024" x2="33.08" y2="16.25" width="0.3" layer="16"/>
-<wire x1="46.8218" y1="15.7024" x2="36.5" y2="15.7024" width="0.3" layer="16"/>
-<wire x1="36.5" y1="15.7024" x2="33.6276" y2="15.7024" width="0.3" layer="16"/>
-<wire x1="36.58" y1="19" x2="36.58" y2="15.7824" width="0.3" layer="16"/>
-<wire x1="36.58" y1="15.7824" x2="36.5" y2="15.7024" width="0.3" layer="16"/>
+<via x="47.05" y="16.4306" extent="1-16" drill="0.35"/>
+<wire x1="47.05" y1="2.65" x2="47.05" y2="16.4306" width="0.3" layer="1"/>
+<wire x1="36.58" y1="19" x2="36.58" y2="16.5" width="0.3" layer="16"/>
+<wire x1="47.05" y1="16.4306" x2="46.9806" y2="16.5" width="0.3" layer="16"/>
+<wire x1="46.9806" y1="16.5" x2="36.58" y2="16.5" width="0.3" layer="16"/>
+<wire x1="36.58" y1="16.5" x2="33.33" y2="16.5" width="0.3" layer="16"/>
+<wire x1="33.33" y1="16.5" x2="33.08" y2="16.25" width="0.3" layer="16"/>
 </signal>
 <signal name="V_TMP">
-<contactref element="U1" pad="ADC"/>
 <contactref element="TMP36" pad="2"/>
-<via x="24.25" y="17.5" extent="1-16" drill="0.35"/>
-<wire x1="24.25" y1="17.5" x2="22.75" y2="17.5" width="0.3" layer="1"/>
-<via x="53" y="15.25" extent="1-16" drill="0.35"/>
-<wire x1="53" y1="15.25" x2="53" y2="19" width="0.3" layer="1"/>
-<wire x1="53" y1="19" x2="53.05" y2="19.05" width="0.3" layer="1"/>
-<wire x1="52.5" y1="14.75" x2="53" y2="15.25" width="0.3" layer="16"/>
-<wire x1="30.875" y1="16.375" x2="32.5" y2="14.75" width="0.3" layer="16"/>
-<wire x1="32.5" y1="14.75" x2="52.5" y2="14.75" width="0.3" layer="16"/>
+<wire x1="32.25" y1="15" x2="30.875" y2="16.375" width="0.3" layer="16"/>
 <wire x1="25.375" y1="16.375" x2="30.875" y2="16.375" width="0.3" layer="16"/>
-<wire x1="24.25" y1="17.5" x2="25.375" y2="16.375" width="0.3" layer="16"/>
-<wire x1="21.5" y1="18.75" x2="20.5" y2="18.75" width="0.3" layer="1"/>
-<wire x1="22.75" y1="17.5" x2="21.5" y2="18.75" width="0.3" layer="1"/>
+<wire x1="25.375" y1="16.375" x2="24.25" y2="17.5" width="0.3" layer="16"/>
+<wire x1="24.25" y1="17.5" x2="21.75" y2="17.5" width="0.3" layer="16"/>
+<wire x1="21.75" y1="17.5" x2="20.5" y2="18.75" width="0.3" layer="16"/>
+<contactref element="SJ1" pad="2"/>
+<wire x1="46.5" y1="14" x2="46.5" y2="14.5" width="0.3" layer="16"/>
+<wire x1="46.5" y1="14.5" x2="45.5" y2="15.5" width="0.3" layer="16"/>
+<wire x1="45.5" y1="15.5" x2="34.25" y2="15.5" width="0.3" layer="16"/>
+<wire x1="34.25" y1="15.5" x2="33.75" y2="15" width="0.3" layer="16"/>
+<wire x1="33.75" y1="15" x2="32.25" y2="15" width="0.3" layer="16"/>
 </signal>
 <signal name="N$2">
@@
 <contactref element="R_GPIO2" pad="2"/>
 <wire x1="45" y1="2.7" x2="45.05" y2="2.65" width="0.3" layer="1"/>
-<wire x1="33.08" y1="11.25" x2="45" y2="11.25" width="0.3" layer="16"/>
-<via x="45" y="11.25" extent="1-16" drill="0.35"/>
-<wire x1="45" y1="11.25" x2="45" y2="2.7" width="0.3" layer="1"/>
+<wire x1="45" y1="10.75" x2="33.58" y2="10.75" width="0.3" layer="16"/>
+<wire x1="33.08" y1="11.25" x2="33.58" y2="10.75" width="0.3" layer="16"/>
+<via x="45" y="10.75" extent="1-16" drill="0.35"/>
+<wire x1="45" y1="10.75" x2="45" y2="2.7" width="0.3" layer="1"/>
 </signal>
 <signal name="PIR">
@@
 <wire x1="11.92" y1="10.25" x2="18.5" y2="10.25" width="0.5" layer="1"/>
 </signal>
-<signal name="N$1">
-<via x="22" y="12.5" extent="1-16" drill="0.35"/>
-</signal>
 <signal name="VDD">
 <contactref element="R_GPIO2" pad="1"/>
 </signal>
+<signal name="TMP_DATA">
+<contactref element="SJ1" pad="3"/>
+<wire x1="44.976" y1="14" x2="43.5" y2="14" width="0.3" layer="16"/>
+<via x="43.5" y="14" extent="1-16" drill="0.35"/>
+</signal>
+<signal name="TMP_ANA">
+<contactref element="SJ1" pad="1"/>
+<wire x1="48.024" y1="14" x2="51.75" y2="14" width="0.3" layer="16"/>
+<wire x1="51.75" y1="14" x2="53" y2="15.25" width="0.3" layer="16"/>
+<via x="53" y="15.25" extent="1-16" drill="0.35"/>
+<contactref element="U1" pad="ADC"/>
+<wire x1="53" y1="19" x2="53.05" y2="19.05" width="0.3" layer="1"/>
+<wire x1="53.05" y1="19.05" x2="53.05" y2="15.3" width="0.3" layer="1"/>
+<wire x1="53.05" y1="15.3" x2="53" y2="15.25" width="0.3" layer="1"/>
+</signal>
+<signal name="N$3">
+<via x="49.75" y="15.75" extent="1-16" drill="0.35"/>
+</signal>
+<signal name="N$4">
+<via x="12.25" y="4.5" extent="1-16" drill="0.35"/>
+</signal>
+<signal name="N$5">
+<via x="7.5" y="5.75" extent="1-16" drill="0.35"/>
+</signal>
 </signals>
