File: hardware/shd_v1.0.sch (EAGLE design)
At the start: 16 parts

Commit message: minor changes and bug fixes
Parts:
- added SJ1: (no value), jumper:SJ2W
Connections:
- new net TMP_ANA: SJ1.1, U1.ADC
- new net TMP_DATA: SJ1.3
- net V_TMP: now also SJ1.2; no longer U1.ADC
Changed lines of the file:
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@@
 <?xml version="1.0" encoding="utf-8"?>
 <!DOCTYPE eagle SYSTEM "eagle.dtd">
-<eagle version="9.2.2">
+<eagle version="9.3.0">
 <drawing>
 <settings>
@@
 <part name="XC6206" library="Voltage Regulator" deviceset="XC6206" device=""/>
 <part name="R_LED_C1" library="eagle-ltspice" library_urn="urn:adsk.eagle:library:217" deviceset="R" device="0207/10" package3d_urn="urn:adsk.eagle:package:13275/1" value="330"/>
+<part name="SJ1" library="jumper" library_urn="urn:adsk.eagle:library:252" deviceset="SJ2W" device="" package3d_urn="urn:adsk.eagle:package:15474/1"/>
 </parts>
 <sheets>
@@
 </segment>
 </net>
-<net name="V_TMP" class="0">
-<segment>
-<pinref part="U1" gate="G$1" pin="ADC"/>
-<wire x1="76.2" y1="83.82" x2="45.72" y2="83.82" width="0.1524" layer="91"/>
-<label x="48.26" y="83.82" size="1.778" layer="95" rot="R180"/>
-</segment>
-</net>
 <net name="N$2" class="0">
 <segment>
@@
 <wire x1="139.7" y1="73.66" x2="147.32" y2="73.66" width="0.1524" layer="91"/>
 <wire x1="147.32" y1="73.66" x2="147.32" y2="76.2" width="0.1524" layer="91"/>
+</segment>
+</net>
+<net name="TMP_ANA" class="0">
+<segment>
+<pinref part="U1" gate="G$1" pin="ADC"/>
+<wire x1="76.2" y1="83.82" x2="45.72" y2="83.82" width="0.1524" layer="91"/>
+<label x="48.26" y="83.82" size="1.778" layer="95" rot="R180"/>
 </segment>
 </net>
@@
 <attribute name="VALUE" x="184.15" y="120.142" size="1.778" layer="96" rot="R180"/>
 </instance>
+<instance part="SJ1" gate="G$1" x="81.28" y="147.32" smashed="yes">
+<attribute name="NAME" x="83.82" y="147.701" size="1.778" layer="95"/>
+<attribute name="VALUE" x="83.82" y="145.415" size="1.778" layer="96"/>
+</instance>
 </instances>
 <busses>
@@
 <segment>
 <pinref part="TMP36" gate="G$1" pin="V_OUT"/>
-<wire x1="50.8" y1="147.32" x2="73.66" y2="147.32" width="0.1524" layer="91"/>
+<wire x1="50.8" y1="147.32" x2="76.2" y2="147.32" width="0.1524" layer="91"/>
 <label x="66.04" y="147.32" size="1.778" layer="95"/>
+<pinref part="SJ1" gate="G$1" pin="2"/>
 </segment>
 </net>
@@
 </segment>
 </net>
+<net name="TMP_DATA" class="0">
+<segment>
+<pinref part="SJ1" gate="G$1" pin="3"/>
+<wire x1="81.28" y1="142.24" x2="81.28" y2="137.16" width="0.1524" layer="91"/>
+<wire x1="81.28" y1="137.16" x2="101.6" y2="137.16" width="0.1524" layer="91"/>
+<label x="93.98" y="137.16" size="1.778" layer="95"/>
+</segment>
+</net>
+<net name="TMP_ANA" class="0">
+<segment>
+<pinref part="SJ1" gate="G$1" pin="1"/>
+<wire x1="81.28" y1="152.4" x2="81.28" y2="157.48" width="0.1524" layer="91"/>
+<wire x1="81.28" y1="157.48" x2="101.6" y2="157.48" width="0.1524" layer="91"/>
+<label x="93.98" y="157.48" size="1.778" layer="95"/>
+</segment>
+</net>
