File: hardware/v2.1/shd_v2.1_double.brd (EAGLE design)
At the start: 69 x 43.8 mm, 25 parts

Commit message: adds hardware v2.1
Parts:
- removed TMP36: TMP36, tmp36:TO-92
- removed U1: (no value), esp8266modules:ESP12E-SMD
- added 10N1: (no value), eagle-ltspice:C0805
- added 5V__LED__GND1, 5V__PIR__GND1: (no value), con-wago-500:W237-103
- added BC1: (no value), transistor:SOT23-BEC
- added DC/DC1: DC-DC-STEP-DOWN-LM2596, diy-modules:DC-DC-STEP-DOWN-LM2596
- added ESP-12E/F, ESP-12E/F1: (no value), esp8266modules:ESP12E-SMD
- added GND__5V1: (no value), con-wago-500:W237-102
- added JP2: (no value), pinhead:1X02
- added PROG_INTERFACE1: (no value), con-lstb:MA05-1
- added R_GPIO1, R_LED_B1: 3k3, eagle-ltspice:0207/10
- added R_LED_C2, R_PROG1, R_RST1: 10k, eagle-ltspice:0207/10
- added R_LED_C3: 330, eagle-ltspice:0207/10
- added SJ10, SJ11, SJ12, SJ13, SJ14: (no value), jumper:SJ
- added SJ8, SJ9: (no value), jumper:SJ_2
- added TMP, TMP1: TMP36, tmp36:TO-92
- added U$2: TEMP-HUM-SENSOR-DHT22, diy-modules:TEMP-HUM-SENSOR-DHT22
- added XC1: (no value), Voltage Regulator:SOT23
- moved U$1 28.5 mm to (18.2, 18.8)
- moved JP1 25.5 mm to (35.0, 5.75), turned to 180 degrees
- moved SJ1 2.25 mm to (48.8, 14.0)
- moved XC6206 1.27 mm to (35.0, 9.25), turned to 90 degrees
- moved BC856 1.12 mm to (35.2, 2.50), turned to 90 degrees
- moved PROG_INTERFACE 1.03 mm to (32.5, 19.0)
- moved 10N 0.25 mm to (35.2, 13.8), turned to 270 degrees
- moved R_RST 0.12 mm to (28.0, 13.8)
- turned R_LED_B to 180 degrees
Connections:
- new net GND1: 10N1.2, 5V__LED__GND1.3, 5V__PIR__GND1.3, BC1.E, ESP-12E/F1.GND, ESP-12E/F1.GPIO15, GND__5V1.2, JP2.1, PROG_INTERFACE1.4, SJ11.1, SJ12.1, SJ13.1, SJ14.1, TMP1.3, U$2.3, U$2.4, XC1.1
- new net GND_STEP_DOWN1: DC/DC1.IN-, DC/DC1.OUT-, SJ11.2, SJ12.2, SJ13.2, SJ14.2
- new net GPIO1: ESP-12E/F1.GPIO0, PROG_INTERFACE1.5, R_PROG1.1
- new net LED_DATA_3.1: ESP-12E/F1.GPIO4, R_LED_B1.2
- new net LED_DATA_3.3_R1: BC1.B, R_LED_B1.1
- new net LED_DATA_5.1: BC1.C, R_LED_C2.1, R_LED_C3.2
- new net LED_DATA_OUT1: 5V__LED__GND1.2, R_LED_C3.1
- new net N$1: ESP-12E/F1.GPIO2, R_GPIO1.2
- new net PIR1: 5V__PIR__GND1.2, ESP-12E/F1.GPIO5
- new net RST1: ESP-12E/F1.RESET, JP2.2, R_RST1.1
- new net RX1: ESP-12E/F1.RXD0, PROG_INTERFACE1.1
- new net TMP_ANA1: ESP-12E/F1.ADC, SJ8.1
- new net TMP_DATA1: ESP-12E/F1.GPIO12, SJ8.3
- new net TX1: ESP-12E/F1.TXD0, PROG_INTERFACE1.2
- new net VCC_5.1: 5V__LED__GND1.1, 5V__PIR__GND1.1, R_LED_C2.2, SJ10.2, SJ9.1, XC1.3
- new net VCC_STEP_DOWN1: DC/DC1.OUT+, SJ10.1
- new net VDD_3.1: 10N1.1, ESP-12E/F1.CH_PD, ESP-12E/F1.VCC, PROG_INTERFACE1.3, R_GPIO1.1, R_PROG1.2, R_RST1.2, TMP1.1, U$2.1, XC1.2
- new net V_IN1: GND__5V1.1, SJ9.2
- new net V_IN_2: DC/DC1.IN+, SJ9.3
- new net V_TMP1: SJ8.2, TMP1.2, U$2.2
- net GND: now also ESP-12E/F.GND, ESP-12E/F.GPIO15, TMP.3; no longer TMP36.3, U1.GND, U1.GPIO15
- net GPIO0: now also ESP-12E/F.GPIO0; no longer U1.GPIO0
- net LED_DATA_3.3: now also ESP-12E/F.GPIO4; no longer U1.GPIO4
- net N$2: now also ESP-12E/F.GPIO2; no longer U1.GPIO2
- net PIR: now also ESP-12E/F.GPIO5; no longer U1.GPIO5
- net RST: now also ESP-12E/F.RESET; no longer U1.RESET
- net RX: now also ESP-12E/F.RXD0; no longer U1.RXD0
- net TMP_ANA: now also ESP-12E/F.ADC; no longer U1.ADC
- net TMP_DATA: now also ESP-12E/F.GPIO12; no longer U$1.2, U1.GPIO12
- net TX: now also ESP-12E/F.TXD0; no longer U1.TXD0
- net VDD_3.3: now also ESP-12E/F.CH_PD, ESP-12E/F.VCC, TMP.1; no longer TMP36.1, U1.CH_PD, U1.VCC
- net V_TMP: now also TMP.2, U$1.2; no longer TMP36.2
Routing:
- net VDD_3.1: track 0.00 -> 67.9 mm, vias 0 -> 2
- net VCC_5.1: track 0.00 -> 63.1 mm, vias 0 -> 2
- net LED_DATA_3.1: track 0.00 -> 60.5 mm, vias 0 -> 4
- net TX1: track 0.00 -> 46.0 mm, vias 0 -> 1
- net RX1: track 0.00 -> 43.8 mm, vias 0 -> 1
- net RST1: track 0.00 -> 40.4 mm, vias 0 -> 1
- net V_TMP1: track 0.00 -> 35.7 mm, vias 0 -> 2
- net PIR1: track 0.00 -> 32.5 mm, vias 0 -> 2
- net GPIO1: track 0.00 -> 27.3 mm
- net LED_DATA_3.3_R1: track 0.00 -> 26.6 mm, vias 0 -> 1
- net LED_DATA_5.1: track 0.00 -> 23.7 mm, vias 0 -> 1
- net V_IN_2: track 0.00 -> 21.5 mm, vias 0 -> 1
- net N$1: track 0.00 -> 18.5 mm, vias 0 -> 1
- net LED_DATA_3.3: track 42.0 -> 60.5 mm, vias 2 -> 4
- net LED_DATA_OUT1: track 0.00 -> 15.6 mm, vias 0 -> 1
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- added copper zone on layer 1, net GND1
- added copper zone on layer 16, net GND1
- added copper zone on layer 16, net GND_STEP_DOWN1
- added copper zone on layer 1, net VCC_STEP_DOWN1
Other:
- board size 69 x 43.8 mm -> 84 x 89.2 mm
- board text added: "3.3V"
- board text added: "GND"
- board text added: "TMP"
